File: PDB.sch (EAGLE design)
At the start: 64 parts, among them IC1 LM555N

Commit message: did initial route of PDB
Parts:
- removed WIPER_SWITCH: (no value), switch:M9040P
- added WIPER_FET: PSMN039-100YS, nxp_60:PSMN039-100YS
- WIPER: value PSMN039-100YS -> (none); device nxp_60:PSMN039-100YS -> switch:M9040P
- renumbered ADD1_SWITCH to ADD_1, ADD2_SWITCH to ADD_2, HAZ_L_SWITCH to HAZ_LEFT, HAZ_R_SWITCH to HAZ_RIGHT
Connections:
- net GND: now also WIPER_FET.S; no longer WIPER.S
- net H4: now also WIPER.O; no longer WIPER_SWITCH.O
- net N$19: now also WIPER_FET.D; no longer WIPER.D
- net N$22: now also WIPER_FET.G; no longer WIPER.G
- net VDD: now also WIPER.P; no longer WIPER_SWITCH.P
Changed lines of the file:
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@@
 <part name="SUPPLY11" library="supply2" library_urn="urn:adsk.eagle:library:372" deviceset="VDD" device=""/>
 <part name="SUPPLY28" library="supply2" library_urn="urn:adsk.eagle:library:372" deviceset="GND" device=""/>
-<part name="WIPER" library="nxp_60" deviceset="PSMN" device="YS" technology="039-100"/>
+<part name="WIPER_FET" library="nxp_60" deviceset="PSMN" device="YS" technology="039-100"/>
 <part name="R9" library="rcl" library_urn="urn:adsk.eagle:library:334" deviceset="R-US_" device="R0805" package3d_urn="urn:adsk.eagle:package:23553/2"/>
 <part name="C10" library="rcl" library_urn="urn:adsk.eagle:library:334" deviceset="C-US" device="C0805" package3d_urn="urn:adsk.eagle:package:23617/2"/>
@@
 <part name="C1" library="rcl" library_urn="urn:adsk.eagle:library:334" deviceset="C-US" device="C0805" package3d_urn="urn:adsk.eagle:package:23617/2" value="33uF"/>
 <part name="R10" library="rcl" library_urn="urn:adsk.eagle:library:334" deviceset="R-US_" device="R0805" package3d_urn="urn:adsk.eagle:package:23553/2" value="1K"/>
-<part name="ADD2_SWITCH" library="switch" library_urn="urn:adsk.eagle:library:380" deviceset="M9040P" device="" package3d_urn="urn:adsk.eagle:package:27676/1"/>
-<part name="ADD1_SWITCH" library="switch" library_urn="urn:adsk.eagle:library:380" deviceset="M9040P" device="" package3d_urn="urn:adsk.eagle:package:27676/1"/>
-<part name="WIPER_SWITCH" library="switch" library_urn="urn:adsk.eagle:library:380" deviceset="M9040P" device="" package3d_urn="urn:adsk.eagle:package:27676/1"/>
-<part name="HAZ_L_SWITCH" library="switch" library_urn="urn:adsk.eagle:library:380" deviceset="M9040P" device="" package3d_urn="urn:adsk.eagle:package:27676/1"/>
-<part name="HAZ_R_SWITCH" library="switch" library_urn="urn:adsk.eagle:library:380" deviceset="M9040P" device="" package3d_urn="urn:adsk.eagle:package:27676/1"/>
+<part name="ADD_2" library="switch" library_urn="urn:adsk.eagle:library:380" deviceset="M9040P" device="" package3d_urn="urn:adsk.eagle:package:27676/1"/>
+<part name="ADD_1" library="switch" library_urn="urn:adsk.eagle:library:380" deviceset="M9040P" device="" package3d_urn="urn:adsk.eagle:package:27676/1"/>
+<part name="WIPER" library="switch" library_urn="urn:adsk.eagle:library:380" deviceset="M9040P" device="" package3d_urn="urn:adsk.eagle:package:27676/1"/>
+<part name="HAZ_LEFT" library="switch" library_urn="urn:adsk.eagle:library:380" deviceset="M9040P" device="" package3d_urn="urn:adsk.eagle:package:27676/1"/>
+<part name="HAZ_RIGHT" library="switch" library_urn="urn:adsk.eagle:library:380" deviceset="M9040P" device="" package3d_urn="urn:adsk.eagle:package:27676/1"/>
 <part name="BRAKE_SNS_OVR" library="switch" library_urn="urn:adsk.eagle:library:380" deviceset="M9040P" device="" package3d_urn="urn:adsk.eagle:package:27676/1"/>
 <part name="REARLIGHTS" library="switch" library_urn="urn:adsk.eagle:library:380" deviceset="M9040P" device="" package3d_urn="urn:adsk.eagle:package:27676/1"/>
@@
 <attribute name="VALUE" x="-29.845" y="-3.175" size="1.778" layer="96"/>
 </instance>
-<instance part="WIPER" gate="G$1" x="12.7" y="5.08" smashed="yes">
+<instance part="WIPER_FET" gate="G$1" x="12.7" y="5.08" smashed="yes">
 <attribute name="NAME" x="11.43" y="10.16" size="1.778" layer="95" font="vector"/>
 </instance>
@@
 <instance part="C1" gate="G$1" x="-20.32" y="104.14"/>
 <instance part="R10" gate="G$1" x="27.94" y="99.06" rot="R270"/>
-<instance part="ADD2_SWITCH" gate="1" x="-66.04" y="-33.02" rot="R270"/>
-<instance part="ADD1_SWITCH" gate="1" x="-30.48" y="-33.02" rot="R270"/>
-<instance part="WIPER_SWITCH" gate="1" x="12.7" y="-33.02" rot="R270"/>
-<instance part="HAZ_L_SWITCH" gate="1" x="53.34" y="-33.02" rot="R270"/>
-<instance part="HAZ_R_SWITCH" gate="1" x="88.9" y="-33.02" rot="R270"/>
+<instance part="ADD_2" gate="1" x="-66.04" y="-33.02" rot="R270"/>
+<instance part="ADD_1" gate="1" x="-30.48" y="-33.02" rot="R270"/>
+<instance part="WIPER" gate="1" x="12.7" y="-33.02" rot="R270"/>
+<instance part="HAZ_LEFT" gate="1" x="53.34" y="-33.02" rot="R270"/>
+<instance part="HAZ_RIGHT" gate="1" x="88.9" y="-33.02" rot="R270"/>
 <instance part="BRAKE_SNS_OVR" gate="1" x="124.46" y="-33.02" rot="R270"/>
 <instance part="REARLIGHTS" gate="1" x="205.74" y="-33.02" rot="R270"/>
@@
 </segment>
 <segment>
-<pinref part="WIPER" gate="G$1" pin="S"/>
+<pinref part="WIPER_FET" gate="G$1" pin="S"/>
 <pinref part="SUPPLY30" gate="GND" pin="GND"/>
 </segment>
@@
 </segment>
 <segment>
-<pinref part="ADD2_SWITCH" gate="1" pin="P"/>
+<pinref part="ADD_2" gate="1" pin="P"/>
 <wire x1="-71.12" y1="-35.56" x2="-73.66" y2="-35.56" width="0.1524" layer="91"/>
 <pinref part="SUPPLY5" gate="G$1" pin="VDD"/>
 </segment>
 <segment>
-<pinref part="ADD1_SWITCH" gate="1" pin="P"/>
+<pinref part="ADD_1" gate="1" pin="P"/>
 <wire x1="-35.56" y1="-35.56" x2="-38.1" y2="-35.56" width="0.1524" layer="91"/>
 <pinref part="SUPPLY6" gate="G$1" pin="VDD"/>
 </segment>
 <segment>
-<pinref part="WIPER_SWITCH" gate="1" pin="P"/>
+<pinref part="WIPER" gate="1" pin="P"/>
 <wire x1="7.62" y1="-35.56" x2="5.08" y2="-35.56" width="0.1524" layer="91"/>
 <pinref part="SUPPLY15" gate="G$1" pin="VDD"/>
@@
 <net name="N$19" class="0">
 <segment>
-<pinref part="WIPER" gate="G$1" pin="D"/>
+<pinref part="WIPER_FET" gate="G$1" pin="D"/>
 <wire x1="15.24" y1="10.16" x2="15.24" y2="17.78" width="0.1524" layer="91"/>
 <pinref part="WIPER_OUT" gate="G$1" pin="GND"/>
@@
 <net name="H3" class="0">
 <segment>
-<pinref part="HAZ_L_SWITCH" gate="1" pin="O"/>
+<pinref part="HAZ_LEFT" gate="1" pin="O"/>
 <wire x1="58.42" y1="-33.02" x2="60.96" y2="-33.02" width="0.1524" layer="91"/>
 <label x="60.96" y="-33.02" size="1.778" layer="95" xref="yes"/>
@@
 <net name="H5" class="0">
 <segment>
-<pinref part="ADD1_SWITCH" gate="1" pin="O"/>
+<pinref part="ADD_1" gate="1" pin="O"/>
 <wire x1="-25.4" y1="-33.02" x2="-20.32" y2="-33.02" width="0.1524" layer="91"/>
 <label x="-20.32" y="-33.02" size="1.778" layer="95" xref="yes"/>
@@
 <net name="H2" class="0">
 <segment>
-<pinref part="HAZ_R_SWITCH" gate="1" pin="O"/>
+<pinref part="HAZ_RIGHT" gate="1" pin="O"/>
 <wire x1="93.98" y1="-33.02" x2="96.52" y2="-33.02" width="0.1524" layer="91"/>
 <label x="96.52" y="-33.02" size="1.778" layer="95" xref="yes"/>
@@
 <net name="H4" class="0">
 <segment>
-<pinref part="WIPER_SWITCH" gate="1" pin="O"/>
+<pinref part="WIPER" gate="1" pin="O"/>
 <wire x1="17.78" y1="-33.02" x2="20.32" y2="-33.02" width="0.1524" layer="91"/>
 <label x="20.32" y="-33.02" size="1.778" layer="95" xref="yes"/>
@@
 <net name="H6" class="0">
 <segment>
-<pinref part="ADD2_SWITCH" gate="1" pin="O"/>
+<pinref part="ADD_2" gate="1" pin="O"/>
 <wire x1="-60.96" y1="-33.02" x2="-58.42" y2="-33.02" width="0.1524" layer="91"/>
 <label x="-58.42" y="-33.02" size="1.778" layer="95" xref="yes"/>
@@
 <net name="555_OUT" class="0">
 <segment>
-<pinref part="HAZ_L_SWITCH" gate="1" pin="P"/>
+<pinref part="HAZ_LEFT" gate="1" pin="P"/>
 <wire x1="48.26" y1="-35.56" x2="45.72" y2="-35.56" width="0.1524" layer="91"/>
 <label x="43.18" y="-38.1" size="1.778" layer="95"/>
 </segment>
 <segment>
-<pinref part="HAZ_R_SWITCH" gate="1" pin="P"/>
+<pinref part="HAZ_RIGHT" gate="1" pin="P"/>
 <wire x1="83.82" y1="-35.56" x2="81.28" y2="-35.56" width="0.1524" layer="91"/>
 <label x="78.74" y="-38.1" size="1.778" layer="95"/>
@@
 <net name="N$22" class="0">
 <segment>
-<pinref part="WIPER" gate="G$1" pin="G"/>
+<pinref part="WIPER_FET" gate="G$1" pin="G"/>
 <pinref part="R14" gate="G$1" pin="2"/>
 <wire x1="10.16" y1="2.54" x2="7.62" y2="2.54" width="0.1524" layer="91"/>
