File: PDB.sch (EAGLE design)
At the start: 77 parts, among them IC1 LM555N

Commit message: changed a lot of routing, near final version with JSTs
Parts:
- removed S1, S2: TL39PO, switch:TL39PO
- added ADD1_, ADD2_: (no value), switch:M9040P
- C10: value (none) -> 22uF; device resistor:EL-BI25-10AXIAL -> SparkFun-Capacitors:22UF-POLAR-PANASONIC_C-35V-20%
Connections:
- net GND: now also C10.-; no longer C10.2
- net H5: now also ADD1_.P; no longer S1.P
- net H6: now also ADD2_.P; no longer S2.P
- net VDD: now also ADD1_.S, ADD2_.S, C10.+; no longer C10.1, S1.S, S2.S
- net µC_1: now also ADD1_.O; no longer S1.O
- net µC_2: now also ADD2_.O; no longer S2.O
Changed lines of the file:
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@@
 <part name="WIPER_" library="nxp_60" deviceset="PSMN" device="YS" technology="039-100"/>
 <part name="R9" library="rcl" library_urn="urn:adsk.eagle:library:334" deviceset="R-US_" device="R0805" package3d_urn="urn:adsk.eagle:package:23553/2"/>
-<part name="C10" library="resistor" library_urn="urn:adsk.eagle:library:348" deviceset="EL-" device="BI25-10AXIAL" package3d_urn="urn:adsk.eagle:package:25992/1"/>
+<part name="C10" library="SparkFun-Capacitors" library_urn="urn:adsk.eagle:library:510" deviceset="22UF-POLAR" device="-PANASONIC_C-35V-20%" package3d_urn="urn:adsk.eagle:package:37430/1" value="22uF"/>
 <part name="GND2" library="supply2" library_urn="urn:adsk.eagle:library:372" deviceset="GND" device=""/>
 <part name="WIPER_OUT" library="powerpoles" deviceset="POWERPOLE_POWER" device="25A_HORIZONTAL_G2" value="POWERPOLE_POWER25A_HORIZONTAL_G2"/>
@@
 <part name="C1" library="rcl" library_urn="urn:adsk.eagle:library:334" deviceset="C-US" device="C0805" package3d_urn="urn:adsk.eagle:package:23617/2" value="33uF"/>
 <part name="R10" library="rcl" library_urn="urn:adsk.eagle:library:334" deviceset="R-US_" device="R0805" package3d_urn="urn:adsk.eagle:package:23553/2" value="1K"/>
-<part name="WIPER" library="switch" library_urn="urn:adsk.eagle:library:380" deviceset="M9040P" device="" package3d_urn="urn:adsk.eagle:package:27676/1"/>
-<part name="HAZ_LEFT" library="switch" library_urn="urn:adsk.eagle:library:380" deviceset="M9040P" device="" package3d_urn="urn:adsk.eagle:package:27676/1"/>
-<part name="HAZ_RIGHT" library="switch" library_urn="urn:adsk.eagle:library:380" deviceset="M9040P" device="" package3d_urn="urn:adsk.eagle:package:27676/1"/>
-<part name="BRAKE_SNS_OVR" library="switch" library_urn="urn:adsk.eagle:library:380" deviceset="M9040P" device="" package3d_urn="urn:adsk.eagle:package:27676/1"/>
-<part name="REARLIGHTS" library="switch" library_urn="urn:adsk.eagle:library:380" deviceset="M9040P" device="" package3d_urn="urn:adsk.eagle:package:27676/1"/>
+<part name="WIPER" library="switch" deviceset="M9040P" device=""/>
+<part name="HAZ_LEFT" library="switch" deviceset="M9040P" device=""/>
+<part name="HAZ_RIGHT" library="switch" deviceset="M9040P" device=""/>
+<part name="BRAKE_SNS_OVR" library="switch" deviceset="M9040P" device=""/>
+<part name="REARLIGHTS" library="switch" deviceset="M9040P" device=""/>
 <part name="SUPPLY7" library="supply2" library_urn="urn:adsk.eagle:library:372" deviceset="VDD" device=""/>
 <part name="SUPPLY15" library="supply2" library_urn="urn:adsk.eagle:library:372" deviceset="VDD" device=""/>
@@
 <part name="SUPPLY21" library="supply2" library_urn="urn:adsk.eagle:library:372" deviceset="GND" device=""/>
 <part name="SUPPLY22" library="supply2" library_urn="urn:adsk.eagle:library:372" deviceset="GND" device=""/>
-<part name="HEADLIGHTS" library="switch" library_urn="urn:adsk.eagle:library:380" deviceset="M9040P" device="" package3d_urn="urn:adsk.eagle:package:27676/1"/>
+<part name="HEADLIGHTS" library="switch" deviceset="M9040P" device=""/>
 <part name="SUPPLY16" library="supply2" library_urn="urn:adsk.eagle:library:372" deviceset="VDD" device=""/>
 <part name="VDD_IN1" library="powerpoles" deviceset="POWERPOLE_POWER" device="25A_HORIZONTAL_G2" value="POWERPOLE_POWER25A_HORIZONTAL_G2"/>
@@
 <part name="J2" library="SparkFun-Connectors" library_urn="urn:adsk.eagle:library:513" deviceset="CONN_05" device="JST" package3d_urn="urn:adsk.eagle:package:38120/1"/>
 <part name="J3" library="SparkFun-Connectors" library_urn="urn:adsk.eagle:library:513" deviceset="CONN_05" device="JST" package3d_urn="urn:adsk.eagle:package:38120/1"/>
-<part name="S1" library="switch" library_urn="urn:adsk.eagle:library:380" deviceset="TL39PO" device="" package3d_urn="urn:adsk.eagle:package:27745/1"/>
-<part name="S2" library="switch" library_urn="urn:adsk.eagle:library:380" deviceset="TL39PO" device="" package3d_urn="urn:adsk.eagle:package:27745/1"/>
 <part name="R15" library="resistor" library_urn="urn:adsk.eagle:library:348" deviceset="R-US_" device="R2512" package3d_urn="urn:adsk.eagle:package:26070/1" value="12K"/>
 <part name="R16" library="resistor" library_urn="urn:adsk.eagle:library:348" deviceset="R-US_" device="R2512" package3d_urn="urn:adsk.eagle:package:26070/1" value="18K"/>
 <part name="SUPPLY5" library="supply2" library_urn="urn:adsk.eagle:library:372" deviceset="GND" device=""/>
+<part name="ADD1_" library="switch" deviceset="M9040P" device=""/>
+<part name="ADD2_" library="switch" deviceset="M9040P" device=""/>
 </parts>
 <sheets>
@@
 <attribute name="VALUE" x="11.938" y="41.91" size="1.778" layer="96" rot="R270"/>
 </instance>
-<instance part="C10" gate="G$1" x="17.78" y="58.42" rot="R90">
-<attribute name="VALUE" x="21.971" y="59.436" size="1.778" layer="96" rot="R90"/>
-</instance>
+<instance part="C10" gate="G$1" x="17.78" y="58.42" rot="R90"/>
 <instance part="GND2" gate="GND" x="22.86" y="55.88"/>
-<instance part="WIPER_OUT" gate="G$1" x="25.4" y="22.86"/>
+<instance part="WIPER_OUT" gate="G$1" x="25.4" y="22.86" smashed="yes">
+<attribute name="NAME" x="20.32" y="30.48" size="1.778" layer="94"/>
+</instance>
 <instance part="SUPPLY29" gate="G$1" x="15.24" y="66.04">
 <attribute name="VALUE" x="13.335" y="69.215" size="1.778" layer="96"/>
@@
 </instance>
 <instance part="GND8" gate="GND" x="22.86" y="45.72"/>
-<instance part="D2" gate="G$1" x="15.24" y="22.86" rot="R90">
+<instance part="D2" gate="G$1" x="15.24" y="22.86" smashed="yes" rot="R90">
+<attribute name="NAME" x="13.335" y="20.574" size="1.778" layer="95" rot="R90"/>
 <attribute name="NAME" x="13.335" y="20.574" size="1.778" layer="95" rot="R90"/>
 </instance>
@@
 <instance part="J2" gate="G$1" x="83.82" y="121.92"/>
 <instance part="J3" gate="G$1" x="114.3" y="144.78"/>
-<instance part="S1" gate="BEF1" x="-27.94" y="-35.56" smashed="yes" rot="R90">
-<attribute name="NAME" x="-25.4" y="-30.48" size="1.778" layer="95" rot="R180"/>
-</instance>
-<instance part="S2" gate="BEF1" x="-66.04" y="-35.56" smashed="yes" rot="R90">
-<attribute name="NAME" x="-63.5" y="-30.48" size="1.778" layer="95" rot="R180"/>
-</instance>
 <instance part="R15" gate="G$1" x="154.94" y="149.86"/>
 <instance part="R16" gate="G$1" x="144.78" y="144.78" rot="R90"/>
 <instance part="SUPPLY5" gate="GND" x="144.78" y="137.16">
 <attribute name="VALUE" x="142.875" y="133.985" size="1.778" layer="96"/>
+</instance>
+<instance part="ADD1_" gate="1" x="-27.94" y="-38.1" rot="R90">
+<attribute name="NAME" x="-26.035" y="-26.67" size="1.778" layer="95" rot="R180"/>
+<attribute name="VALUE" x="-30.48" y="-41.91" size="1.778" layer="96" rot="R180"/>
+</instance>
+<instance part="ADD2_" gate="1" x="-66.04" y="-38.1" rot="R90">
+<attribute name="NAME" x="-64.135" y="-26.67" size="1.778" layer="95" rot="R180"/>
+<attribute name="VALUE" x="-68.58" y="-41.91" size="1.778" layer="96" rot="R180"/>
 </instance>
 </instances>
@@
 <segment>
 <pinref part="GND2" gate="GND" pin="GND"/>
-<pinref part="C10" gate="G$1" pin="2"/>
+<pinref part="C10" gate="G$1" pin="-"/>
 </segment>
 <segment>
@@
 <pinref part="SUPPLY29" gate="G$1" pin="VDD"/>
 <wire x1="15.24" y1="63.5" x2="15.24" y2="58.42" width="0.1524" layer="91"/>
-<pinref part="C10" gate="G$1" pin="1"/>
+<pinref part="C10" gate="G$1" pin="+"/>
 <junction x="15.24" y="58.42"/>
 <pinref part="R9" gate="G$1" pin="1"/>
@@
 </segment>
 <segment>
-<pinref part="S2" gate="BEF1" pin="S"/>
 <wire x1="-71.12" y1="-33.02" x2="-73.66" y2="-33.02" width="0.1524" layer="91"/>
 <label x="-76.2" y="-33.02" size="1.016" layer="95"/>
-</segment>
-<segment>
-<pinref part="S1" gate="BEF1" pin="S"/>
+<pinref part="ADD2_" gate="1" pin="S"/>
+</segment>
+<segment>
 <wire x1="-33.02" y1="-33.02" x2="-35.56" y2="-33.02" width="0.1524" layer="91"/>
 <label x="-38.1" y="-33.02" size="1.016" layer="95"/>
+<pinref part="ADD1_" gate="1" pin="S"/>
 </segment>
 </net>
@@
 </segment>
 <segment>
-<pinref part="S1" gate="BEF1" pin="P"/>
 <wire x1="-22.86" y1="-35.56" x2="-17.78" y2="-35.56" width="0.1524" layer="91"/>
 <label x="-15.24" y="-35.56" size="1.016" layer="95"/>
+<pinref part="ADD1_" gate="1" pin="P"/>
 </segment>
 </net>
@@
 </segment>
 <segment>
-<pinref part="S2" gate="BEF1" pin="P"/>
 <wire x1="-60.96" y1="-35.56" x2="-55.88" y2="-35.56" width="0.1524" layer="91"/>
 <label x="-53.34" y="-35.56" size="1.016" layer="95"/>
+<pinref part="ADD2_" gate="1" pin="P"/>
 </segment>
 </net>
@@
 </segment>
 <segment>
-<pinref part="S2" gate="BEF1" pin="O"/>
 <wire x1="-71.12" y1="-38.1" x2="-73.66" y2="-38.1" width="0.1524" layer="91"/>
 <label x="-76.2" y="-38.1" size="1.016" layer="95"/>
+<pinref part="ADD2_" gate="1" pin="O"/>
 </segment>
 </net>
@@
 </segment>
 <segment>
-<pinref part="S1" gate="BEF1" pin="O"/>
 <wire x1="-33.02" y1="-38.1" x2="-35.56" y2="-38.1" width="0.1524" layer="91"/>
 <label x="-38.1" y="-38.1" size="1.016" layer="95"/>
-</segment>
-</net>
+<pinref part="ADD1_" gate="1" pin="O"/>
+</segment>
+</net>

Commit message: updated PDB board
Parts:
- D1: device diode:ZENER-DIODEDO34-7 -> diode:ZENER-DIODEDO41Z10
- D2: value 1N5817-B -> 1N4446; device diode:1N5817-B -> diode:1N4446
- R1, R2, R20, R21, R3, R4, R5, R6: value 10K -> 510
- R15, R16: device resistor:R-US_R2512 -> resistor:R-US_R3225

Commit message: added Molex for MC signals
Parts:
- removed J1, J2, J3: (no value), SparkFun-Connectors:CONN_05JST
- removed R7, R8: 0, rcl:R-US_R0805
- removed R9: (no value), rcl:R-US_R0805
- added ADD_IN, SPI_IN, SPI_OUT: 8-PIN-MOLEX-RA-FEMALE, master_library:8-PIN-MOLEX-RA-FEMALE
Connections:
- removed net N$12: J2.5
- removed net N$16: ADD2_OUT.V+, R7.2
- removed net N$20: D2.C, R9.2, WIPER_OUT.V+
- net BRK_SNS_5V: now also ADD_IN.P$1, SPI_IN.P$1; no longer J1.5, J3.5
- net CS_SPI: now also SPI_IN.P$4, SPI_OUT.P$4; no longer J1.2, J2.2
- net GND: now also SPI_OUT.P$6
- net MISO_SPI: now also SPI_IN.P$2, SPI_OUT.P$2; no longer J1.4, J2.4
- net MOSI_SPI: now also SPI_IN.P$3, SPI_OUT.P$3; no longer J1.3, J2.3
- net N$18: now also SPI_IN.P$6; no longer ADD1_OUT.V+, R8.2
- net SCL_SPI: now also SPI_IN.P$5, SPI_OUT.P$5; no longer J1.1, J2.1
- net VDD: now also ADD1_OUT.V+, ADD2_OUT.V+, D2.C, SPI_OUT.P$1, WIPER_OUT.V+; no longer R7.1, R8.1, R9.1
- net µC_1: now also ADD_IN.P$3; no longer J3.3
- net µC_2: now also ADD_IN.P$2; no longer J3.4
Other:
- moved on the sheet: R15, R16, VDD_IN, VDD_IN1
