File: big_picture.brd (EAGLE design)
At the start: 160 x 100 mm, 11 parts, among them K1 RELAY-SPDT-JZC-11F, M1 MOTOR10MM

Commit message: did initial route of PDB
Parts:
- added F3, FUSE_3A, FUSE_40A: FUSESH22,5A, fuse:SH22,5A
Connections:
- removed net N$1: E_STOP1.2
- new net FUSE_10A: E_STOP1.2, F3.1, F3.2
- net N$32: now also FUSE_3A.1, FUSE_3A.2, FUSE_40A.1, FUSE_40A.2
Changed lines of the file:
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@@
 <attribute name="SF_SKU" value="ROB-08449" x="-139.7" y="-195.58" size="1.778" layer="27" display="off"/>
+</element>
+<element name="FUSE_3A" library="fuse" library_urn="urn:adsk.eagle:library:233" package="SH22,5A" package3d_urn="urn:adsk.eagle:package:14070/1" value="FUSESH22,5A" x="-127" y="-207.01">
+<attribute name="MF" value="" x="-127" y="-207.01" size="1.4224" layer="27" display="off"/>
+<attribute name="MPN" value="" x="-127" y="-207.01" size="1.4224" layer="27" display="off"/>
+<attribute name="OC_FARNELL" value="unknown" x="-127" y="-207.01" size="1.4224" layer="27" display="off"/>
+<attribute name="OC_NEWARK" value="unknown" x="-127" y="-207.01" size="1.4224" layer="27" display="off"/>
+</element>
+<element name="FUSE_40A" library="fuse" library_urn="urn:adsk.eagle:library:233" package="SH22,5A" package3d_urn="urn:adsk.eagle:package:14070/1" value="FUSESH22,5A" x="-127" y="-220.98">
+<attribute name="MF" value="" x="-127" y="-220.98" size="1.4224" layer="27" display="off"/>
+<attribute name="MPN" value="" x="-127" y="-220.98" size="1.4224" layer="27" display="off"/>
+<attribute name="OC_FARNELL" value="unknown" x="-127" y="-220.98" size="1.4224" layer="27" display="off"/>
+<attribute name="OC_NEWARK" value="unknown" x="-127" y="-220.98" size="1.4224" layer="27" display="off"/>
+</element>
+<element name="F3" library="fuse" library_urn="urn:adsk.eagle:library:233" package="SH22,5A" package3d_urn="urn:adsk.eagle:package:14070/1" value="FUSESH22,5A" x="-127" y="-234.95">
+<attribute name="MF" value="" x="-127" y="-234.95" size="1.4224" layer="27" display="off"/>
+<attribute name="MPN" value="" x="-127" y="-234.95" size="1.4224" layer="27" display="off"/>
+<attribute name="OC_FARNELL" value="unknown" x="-127" y="-234.95" size="1.4224" layer="27" display="off"/>
+<attribute name="OC_NEWARK" value="unknown" x="-127" y="-234.95" size="1.4224" layer="27" display="off"/>
 </element>
 </elements>
@@
 <contactref element="K1" pad="3"/>
 <contactref element="S1" pad="2"/>
+<contactref element="FUSE_3A" pad="2"/>
+<contactref element="FUSE_3A" pad="1"/>
+<contactref element="FUSE_40A" pad="2"/>
+<contactref element="FUSE_40A" pad="1"/>
 <wire x1="-127" y1="-83.82" x2="-115.57" y2="-100.33" width="0" layer="19" extent="1-1"/>
 <wire x1="-134.62" y1="-128.27" x2="-115.57" y2="-100.33" width="0" layer="19" extent="1-1"/>
+<wire x1="-138.2522" y1="-207.01" x2="-134.62" y2="-128.27" width="0" layer="19" extent="1-1"/>
+<wire x1="-138.2522" y1="-220.98" x2="-138.2522" y2="-207.01" width="0" layer="19" extent="1-1"/>
+<wire x1="-115.7478" y1="-220.98" x2="-138.2522" y2="-220.98" width="0" layer="19" extent="1-1"/>
+<wire x1="-115.7478" y1="-207.01" x2="-115.7478" y2="-220.98" width="0" layer="19" extent="1-1"/>
 </signal>
 <signal name="N$35">
@@
 <wire x1="-132.08" y1="-128.27" x2="-127" y2="-88.9" width="0" layer="19" extent="1-1"/>
 </signal>
-<signal name="N$1">
+<signal name="FUSE_10A">
 <contactref element="E_STOP1" pad="2"/>
+<contactref element="F3" pad="2"/>
+<contactref element="F3" pad="1"/>
+<wire x1="-115.7478" y1="-234.95" x2="-138.2522" y2="-234.95" width="0" layer="19" extent="1-1"/>
+<wire x1="-133.35" y1="-154.94" x2="-138.2522" y2="-234.95" width="0" layer="19" extent="1-1"/>
 </signal>
 <signal name="N$3">
